Commit message: added arm and gripper parameters

File: paul/paul_description/urdf/arms/gen3_lite_gen3_lite_2f.xacro (robot description, xacro)
@@ -1,6 +1,3 @@
 <?xml version="1.0"?>
-<!-- Modified version of gen3_lite_gen3_lite_2f.xacro from kortex_description -->
-<!-- Olivier Roy - 2022-01-17 -->
-<!-- PMC-Paul -->
 <robot name="gen3_lite_gen3_lite_2f" xmlns:xacro="http://ros.org/wiki/xacro">
     <!-- Arguments -->
@@ -11,5 +8,5 @@
     <xacro:arg name="gripper" default="gen3_lite_2f" />
     <xacro:arg name="sim" default="false" />
-    <xacro:arg name="prefix" default="gen3_lite_" />
+    <xacro:arg name="prefix" default="$(arg arm)_$(arg gripper)_" />
     <xacro:include filename="$(find kortex_description)/robots/kortex_robot.xacro" />
     <xacro:load_robot arm="$(arg arm)" gripper="$(arg gripper)" dof="$(arg dof)" vision="false" sim="$(arg sim)"  prefix="$(arg prefix)" />

File: paul/paul_description/urdf/paul.urdf.xacro (robot description, xacro)
@@ -4,4 +4,7 @@
   based on https://answers.ros.org/question/379014/passing-outside-parameters-into-urdf-file-using-xacro/ -->
   <xacro:arg name="simulation" default="true"/>
+  <!-- Kinova arm parameters -->
+  <xacro:arg name="arm"        default="gen3_lite"/>
+  <xacro:arg name="gripper"    default="gen3_lite_2f"/>
   <!-- Need seperate property for xacro inorder processing -->
   <xacro:property name="simulation" value="$(arg simulation)"/>
@@ -64,5 +67,5 @@
   <xacro:include filename="$(find paul_description)/urdf/paul.gazebo.xacro" />
   <xacro:include filename="$(find paul_description)/urdf/sensors/lidar.urdf.xacro" />
-  <xacro:include filename="$(find paul_description)/urdf/arms/gen3_lite.urdf.xacro" />
+  <xacro:include filename="$(find paul_description)/urdf/arms/$(arg arm)_$(arg gripper).xacro"/>
   <xacro:include filename="$(find paul_description)/urdf/d435/_d435.urdf.xacro"/>
   <!-- BASE FOOTPRINT -->
@@ -139,5 +142,5 @@
   <joint name="baseArm" type="fixed">
     <parent link="linearAxis_link"/>
-    <child link="gen3_lite_base_link"/>
+    <child link="$(arg arm)_$(arg gripper)_base_link"/>
     <origin xyz="0.0 0.0 0.0" rpy="0 1.5708 0"/>
   </joint>
