Commit message: Refactor: - Modified launch files in bringup to use with paul_gazebo - Modified URDF to only include arm in real life - Added arm.launch to use arm without cart in sim and real life

File: paul/paul_description/urdf/arms/arm.xacro (robot description, xacro)
@@ -1,13 +1,16 @@
 <?xml version="1.0"?>
-<robot name="gen3_lite_gen3_lite_2f" xmlns:xacro="http://ros.org/wiki/xacro">
+<robot name="arm" xmlns:xacro="http://ros.org/wiki/xacro">
     <!-- Arguments -->
     <xacro:arg name="arm" default="gen3_lite" />
-    <!-- Those arguments are ignored for now on Gen3 lite because there is only one supported configuration -->
     <xacro:arg name="dof" default="6" />
     <xacro:arg name="vision" default="false" />
     <xacro:arg name="gripper" default="gen3_lite_2f" />
     <xacro:arg name="sim" default="false" />
-    <xacro:arg name="prefix" default="$(arg arm)_$(arg gripper)_" />
-    <xacro:include filename="$(find paul_description)/urdf/arms/kortex_robot.xacro" />
-    <xacro:load_robot arm="$(arg arm)" gripper="$(arg gripper)" dof="$(arg dof)" vision="false" sim="$(arg sim)"  prefix="$(arg prefix)" />
+    <xacro:include filename="$(find kortex_description)/robots/kortex_robot.xacro" />
+    <xacro:load_robot arm="$(arg arm)" gripper="$(arg gripper)" dof="$(arg dof)" vision="$(arg vision)" sim="$(arg sim)"  prefix="arm_" />
+    <joint name="arm_mount" type="fixed">
+        <parent link="linear_axis_link"/>
+        <child link="arm_base_link"/>
+        <origin xyz="0.0 0.0 0.0" rpy="0.0 0.0 0.0"/>
+    </joint>
 </robot>

File: paul/paul_description/urdf/paul.urdf.xacro (robot description, xacro)
@@ -1,16 +1,15 @@
 <?xml version="1.0"?>
 <robot name="paul" xmlns:xacro="http://www.ros.org/wiki/xacro">
+  <!-- ============================================== -->
+  <!-- ================= PARAMETERS ================= -->
+  <!-- ============================================== -->
   <!-- Need argument to get from launch file:
   based on https://answers.ros.org/question/379014/passing-outside-parameters-into-urdf-file-using-xacro/ -->
-  <xacro:arg name="sim" default="true"/>
+  <xacro:arg name="sim" default="false"/>
   <!-- Kinova arm parameters -->
-  <xacro:arg name="arm"     default="$(optenv PAUL_ARM_MODEL gen3_lite)" />
-  <xacro:arg name="dof"     default="$(optenv PAUL_ARM_DOF 6)" />
-  <xacro:arg name="vision"  default="$(optenv PAUL_ARM_VISION false)" />
-  <xacro:arg name="gripper" default="$(optenv PAUL_ARM_GRIPPER gen3_lite_2f)" />
-  <xacro:arg name="sim"     default="$(optenv PAUL_ARM_SIM false)" />
-  <xacro:arg name="prefix"  default="$(optenv PAUL_ARM_PREFIX arm_)" />
-  <!-- Need seperate property for xacro inorder processing -->
-  <xacro:property name="sim" value="$(arg sim)"/>
+  <xacro:arg name="arm"     default="gen3"/>
+  <xacro:arg name="dof"     default="7"/>
+  <xacro:arg name="vision"  default="true"/>
+  <xacro:arg name="gripper" default=""/>
   <!-- Constant for paul base -->
   <xacro:property name="mass" 			value="20.0" />
@@ -59,5 +58,5 @@
   <xacro:property name="caster_L_rot_y"		value=" ${caster_R_rot_y}"/>
   <xacro:property name="caster_L_rot_z"		value=" ${caster_R_rot_z}"/>
-  <!-- RGBD Sensor parameters -->
+  <!-- RGBD sensor parameters -->
   <xacro:property name="realsense_pose_x" value="${base_width}" />
   <xacro:property name="realsense_pose_y" value="0.0" />
@@ -67,4 +66,7 @@
   <xacro:property name="realsense_rot_y" value="0.0" />
   <xacro:property name="realsense_rot_z" value="0.0" />
+  <!-- ============================================== -->
+  <!-- ================= COMPONENTS ================= -->
+  <!-- ============================================== -->
   <!-- Included files -->
   <xacro:include filename="$(find paul_description)/urdf/components/wheel.urdf.xacro" />
@@ -72,10 +74,11 @@
   <xacro:include filename="$(find paul_description)/urdf/paul.gazebo.xacro" />
   <xacro:include filename="$(find paul_description)/urdf/sensors/lidar.urdf.xacro" />
-  <xacro:include filename="$(find paul_description)/urdf/d435/_d435.urdf.xacro"/>
-  <xacro:include filename="$(find paul_description)/urdf/arms/paul_gen3_lite_description.urdf.xacro" />
-  <!-- BASE FOOTPRINT -->
+  <xacro:include filename="$(find paul_description)/urdf/sensors/d435/_d435.urdf.xacro"/>
+  <!-- ============================================== -->
+  <!-- ==================== BASE ==================== -->
+  <!-- ============================================== -->
   <!-- base_footprint is a fictitious link(frame) that is on the ground right below base_link origin -->
   <link name="base_footprint"/>
-  <!-- BASE_LINK (only static pieces) -->
+  <!-- base_link (only static pieces) -->
   <link name="base_link">
     <inertial>
@@ -107,4 +110,17 @@
     <origin xyz="0.0 0.0 ${ground_to_base_z}" rpy="0 0 0"/>
   </joint>
+  <!-- driven wheels -->
+    <!-- Right Wheel: "wheel_R_link" and "wheel_R_joint" -->
+  <xacro:wheel lr="R" parent="base_link" wheelRadius="${wheel_radius}" wheelLength="${wheel_thickness}" wheelMass="${wheel_mass}" posX="${wheel_R_pose_x}" posY="${wheel_R_pose_y}" posZ="${wheel_R_pose_z}" flipY="1"/>
+    <!-- Left Wheel: "wheel_L_link" and "wheel_L_joint" -->
+  <xacro:wheel lr="L" parent="base_link" wheelRadius="${wheel_radius}" wheelLength="${wheel_thickness}" wheelMass="${wheel_mass}" posX="${wheel_L_pose_x}" posY="${wheel_L_pose_y}" posZ="${wheel_L_pose_z}" flipY="1"/>
+  <!-- caster wheels -->
+    <!-- Right caster wheel: "caster_R_link" and "caster_R_joint" -->
+  <xacro:caster lr="R" parent="base_link" casterRadius="${wheel_radius}" casterMass="${wheel_mass}" posX="${caster_R_pose_x}" posY="${caster_R_pose_y}" posZ="${caster_R_pose_z}" flipY="1"/>
+    <!-- Left caster wheel: "caster_L_link" and "caster_L_joint" -->
+  <xacro:caster lr="L" parent="base_link" casterRadius="${wheel_radius}" casterMass="${wheel_mass}" posX="${caster_L_pose_x}" posY="${caster_L_pose_y}" posZ="${caster_L_pose_z}" flipY="1"/>
+  <!-- ============================================== -->
+  <!-- ================== SENSORS =================== -->
+  <!-- ============================================== -->
   <!-- IMU -->
   <link name="imu_link"/>
@@ -135,29 +151,4 @@
     <origin xyz="0 0 0" rpy="0 0 0"/>
   </joint>
-  <!-- Arm linear axis -->
-  <link name="linearAxis_link" />
-  <joint name="linearAxis" type="prismatic">
-    <limit effort="1000.0" lower="0" upper="1" velocity="0.5"/>
-    <parent link="base_link"/>
-    <child link="linearAxis_link"/>
-    <origin xyz="-0.6 0.0 0.0" rpy="0 -1.5708 0"/>
-  </joint>
-  <link name="armMount_link"/>
-  <joint name="armMount" type="fixed">
-    <parent link="linearAxis_link"/>
-    <child link="armMount_link"/>
-    <origin xyz="0.0 0.0 0.0" rpy="0.0 0.0 0.0"/>
-  </joint>
-  <xacro:include filename="$(find paul_description)/urdf/arms/arm.xacro"/> -->
-  <!-- driven wheels -->
-    <!-- Right Wheel: "wheel_R_link" and "wheel_R_joint" -->
-  <xacro:wheel lr="R" parent="base_link" wheelRadius="${wheel_radius}" wheelLength="${wheel_thickness}" wheelMass="${wheel_mass}" posX="${wheel_R_pose_x}" posY="${wheel_R_pose_y}" posZ="${wheel_R_pose_z}" flipY="1"/>
-    <!-- Left Wheel: "wheel_L_link" and "wheel_L_joint" -->
-  <xacro:wheel lr="L" parent="base_link" wheelRadius="${wheel_radius}" wheelLength="${wheel_thickness}" wheelMass="${wheel_mass}" posX="${wheel_L_pose_x}" posY="${wheel_L_pose_y}" posZ="${wheel_L_pose_z}" flipY="1"/>
-  <!-- caster wheels -->
-    <!-- Right caster wheel: "caster_R_link" and "caster_R_joint" -->
-  <xacro:caster lr="R" parent="base_link" casterRadius="${wheel_radius}" casterMass="${wheel_mass}" posX="${caster_R_pose_x}" posY="${caster_R_pose_y}" posZ="${caster_R_pose_z}" flipY="1"/>
-    <!-- Left caster wheel: "caster_L_link" and "caster_L_joint" -->
-  <xacro:caster lr="L" parent="base_link" casterRadius="${wheel_radius}" casterMass="${wheel_mass}" posX="${caster_L_pose_x}" posY="${caster_L_pose_y}" posZ="${caster_L_pose_z}" flipY="1"/>
   <!-- Lidar sensor -->
   <xacro:lidar parent="base_link">
@@ -165,6 +156,29 @@
   </xacro:lidar>
   <!-- D435 RGB-D Sensor -->
-  <xacro:sensor_d435 parent="base_link" use_nominal_extrinsics="${sim}">
+  <xacro:sensor_d435 parent="base_link" use_nominal_extrinsics="${use_nominal_extrinsics}">
     <origin xyz="${realsense_pose_x} ${realsense_pose_y} ${realsense_pose_z}" rpy="${realsense_rot_x} ${realsense_rot_y} ${realsense_rot_z}"/>
   </xacro:sensor_d435>
+  <!-- ============================================== -->
+  <!-- ==================== ARM ===================== -->
+  <!-- ============================================== -->
+  <xacro:unless value="$(arg sim)">
+    <!-- linear axis -->
+    <link name="linear_axis_link" />
+    <joint name="linear_axis" type="prismatic">
+      <limit effort="1000.0" lower="0" upper="1" velocity="0.5"/>
+      <axis xyz="0 0 1"/>
+      <parent link="base_link"/>
+      <child link="linear_axis_link"/>
+      <origin xyz="-0.6 0.0 0.0" rpy="0 0 0"/>
+    </joint>
+    <!-- load arm -->
+    <xacro:include filename="$(find paul_description)/urdf/arms/kortex_robot.xacro" />
+    <xacro:load_robot arm="$(arg arm)" gripper="$(arg gripper)" dof="$(arg dof)" vision="$(arg vision)" sim="$(arg sim)"  prefix="arm_" />
+    <!-- attach arm to newly created link -->
+    <joint name="arm_mount" type="fixed">
+      <parent link="linear_axis_link"/>
+      <child link="arm_base_link"/>
+      <origin xyz="0.0 0.0 0.0" rpy="0.0 0.0 0.0"/>
+    </joint>
+  </xacro:unless>
 </robot>

File: paul/paul_description/urdf/sensors/d435/_d435.urdf.xacro (robot description, xacro)
@@ -12,6 +12,6 @@
 <robot name="sensor_d435" xmlns:xacro="http://ros.org/wiki/xacro">
   <!-- Includes -->
-  <xacro:include filename="$(find paul_description)/urdf/d435/_d435.gazebo.xacro"/>
-  <xacro:include filename="$(find paul_description)/urdf/d435/_usb_plug.urdf.xacro" />
+  <xacro:include filename="$(find paul_description)/urdf/sensors/d435/_d435.gazebo.xacro"/>
+  <xacro:include filename="$(find paul_description)/urdf/sensors/d435/_usb_plug.urdf.xacro" />
   <xacro:macro name="sensor_d435" params="parent *origin name:=camera topics_ns:=camera use_nominal_extrinsics:=false add_plug:=false use_mesh:=true publish_pointcloud:=true">
     <xacro:property name="M_PI" value="3.1415926535897931" />

File: paul/paul_description/urdf/sensors/lidar.urdf.xacro (robot description, xacro)
@@ -10,11 +10,11 @@
             <visual>
                 <geometry>
-                    <box size ="0.1 0.1 0.1" />
-                    <!--mesh filename="package://paul_description/meshes/lidar.stl" /-->
+                    <cylinder length="0.05" radius="0.05"/>
+                    <!-- <mesh filename="package://paul_description/meshes/lidar.stl" scale="0.001 0.001 0.001"/> -->
                 </geometry>
             </visual>
             <collision>
                 <geometry>
-                    <box size="0.1 0.1 0.1"/>
+                    <cylinder length="0.05" radius="0.05"/>
                 </geometry>
             </collision>
@@ -47,5 +47,5 @@
                 <plugin name="laser_node" filename="libgazebo_ros_laser.so">
                     <topicName>/laser_scan</topicName>
-                    <frameName>laser_link</frameName>
+                    <frameName>/laser_link</frameName> <!-- slash required for global namespace -->
                 </plugin>
             </sensor>
