Commit message: fixed namespace issues and mapping

File: paul/paul_description/urdf/components/wheel.urdf.xacro (robot description, xacro)
@@ -44,4 +44,23 @@
       </inertial>
     </link>
+    <joint name="wheel_${lr}_joint" type="continuous">
+      <parent link="${parent}"/>
+      <child link="wheel_${lr}_link"/>
+      <origin xyz="${posX} ${posY} ${posZ}" rpy="0 0 0" />
+      <axis xyz="0 1 0" rpy="0  0" />
+      <limit effort="100" velocity="100"/>
+      <joint_properties damping="0.0" friction="0.0"/>
+    </joint>
+    <!-- Transmission is important to link the joints and the controller -->
+    <transmission name="wheel_${lr}_joint_trans">
+      <type>transmission_interface/SimpleTransmission</type>
+      <joint name="wheel_${lr}_joint">
+        <hardwareInterface>EffortJointInterface</hardwareInterface>
+      </joint>
+      <actuator name="wheel_${lr}_joint_motor">
+        <hardwareInterface>EffortJointInterface</hardwareInterface>
+        <mechanicalReduction>1</mechanicalReduction>
+      </actuator>
+    </transmission>
     <gazebo reference="wheel_${lr}_link">
       <mu1 value="1.0"/>
@@ -53,21 +72,4 @@
       <turnGravityOff>false</turnGravityOff>
     </gazebo>
-    <joint name="wheel_${lr}_joint" type="continuous">
-      <parent link="${parent}"/>
-      <child link="wheel_${lr}_link"/>
-      <origin xyz="${posX} ${posY} ${posZ}" rpy="0 0 0" />
-      <axis xyz="0 1 0" rpy="0  0" />
-      <limit effort="100" velocity="100"/>
-      <joint_properties damping="0.0" friction="0.0"/>
-    </joint>
-    <!-- Transmission is important to link the joints and the controller -->
-    <transmission name="$wheel_${lr}_joint_trans">
-      <type>transmission_interface/SimpleTransmission</type>
-      <joint name="$wheel_${lr}_joint" />
-      <actuator name="$wheel_${lr}_joint_motor">
-        <hardwareInterface>EffortJointInterface</hardwareInterface>
-        <mechanicalReduction>1</mechanicalReduction>
-      </actuator>
-    </transmission>
   </xacro:macro>
 </robot>

File: paul/paul_description/urdf/paul.gazebo.xacro (robot description, xacro)
@@ -12,6 +12,6 @@
       <rosDebugLevel>na</rosDebugLevel>
       <publishWheelTF>false</publishWheelTF>
-      <robotNamespace>/</robotNamespace>
       <publishTf>1</publishTf>
+      <publish_odom>1</publish_odom>
       <publishWheelJointState>false</publishWheelJointState>
       <alwaysOn>true</alwaysOn>
@@ -27,5 +27,5 @@
       <odometryFrame>odom</odometryFrame>
       <odometryTopic>odom</odometryTopic>
-      <robotBaseFrame>base_footprint</robotBaseFrame>
+      <robotBaseFrame>/base_footprint</robotBaseFrame>
     </plugin>
   </gazebo>

File: paul/paul_description/urdf/paul.urdf.xacro (robot description, xacro)
@@ -156,5 +156,5 @@
   </xacro:lidar>
   <!-- D435 RGB-D Sensor -->
-  <xacro:sensor_d435 parent="base_link" use_nominal_extrinsics="${use_nominal_extrinsics}">
+  <xacro:sensor_d435 parent="base_link" use_nominal_extrinsics="${use_nominal_extrinsics}" name="realsense" topics_ns="realsense">
     <origin xyz="${realsense_pose_x} ${realsense_pose_y} ${realsense_pose_z}" rpy="${realsense_rot_x} ${realsense_rot_y} ${realsense_rot_z}"/>
   </xacro:sensor_d435>

File: paul/paul_description/urdf/sensors/d435/_d435.urdf.xacro (robot description, xacro)
@@ -14,5 +14,5 @@
   <xacro:include filename="$(find paul_description)/urdf/sensors/d435/_d435.gazebo.xacro"/>
   <xacro:include filename="$(find paul_description)/urdf/sensors/d435/_usb_plug.urdf.xacro" />
-  <xacro:macro name="sensor_d435" params="parent *origin name:=camera topics_ns:=camera use_nominal_extrinsics:=false add_plug:=false use_mesh:=true publish_pointcloud:=true">
+  <xacro:macro name="sensor_d435" params="parent *origin name:=realsense topics_ns:=realsense use_nominal_extrinsics:=false add_plug:=false use_mesh:=true publish_pointcloud:=true">
     <xacro:property name="M_PI" value="3.1415926535897931" />
     <!-- The following values are approximate, and the camera node
