Commit message: mapping working

File: paul/paul_description/urdf/components/caster.urdf.xacro (robot description, xacro)
@@ -51,5 +51,5 @@
     </gazebo>
     <!--Joint definition-->
-    <joint name="caster_${lr}_joint" type="continuous">
+    <joint name="caster_${lr}_joint" type="fixed">
       <parent link="${parent}"/>
       <child link="caster_${lr}_link"/>
