Commit message: Added Lidar and front camera. Started designing map.

File: paul/paul_description/urdf/paul.gazebo.xacro (robot description, xacro)
@@ -22,5 +22,5 @@
       <wheelDiameter>${2*wheel_radius}</wheelDiameter>
       <broadcastTF>1</broadcastTF>
-      <wheelTorque>30</wheelTorque>
+      <wheelTorque>100</wheelTorque>
       <wheelAcceleration>1.8</wheelAcceleration>
       <commandTopic>cmd_vel</commandTopic>
@@ -30,3 +30,42 @@
     </plugin>
   </gazebo>
+  <gazebo reference="rgb1_link">
+    <sensor type="camera" name="camera1">
+      <update_rate>30.0</update_rate>
+      <camera name="rgb1">
+        <horizontal_fov>1.3962634</horizontal_fov>
+        <image>
+          <width>800</width>
+          <height>800</height>
+          <format>R8G8B8</format>
+        </image>
+        <clip>
+          <near>0.02</near>
+          <far>300</far>
+        </clip>
+        <noise>
+          <type>gaussian</type>
+          <!-- Noise is sampled independently per pixel on each frame.
+               That pixel's noise value is added to each of its color
+               channels, which at that point lie in the range [0,1]. -->
+          <mean>0.0</mean>
+          <stddev>0.007</stddev>
+        </noise>
+      </camera>
+      <plugin name="camera_controller" filename="libgazebo_ros_camera.so">
+        <alwaysOn>true</alwaysOn>
+        <updateRate>0.0</updateRate>
+        <cameraName>camera1</cameraName>
+        <imageTopicName>image_raw</imageTopicName>
+        <cameraInfoTopicName>camera_info</cameraInfoTopicName>
+        <frameName>rgb1_link</frameName>
+        <hackBaseline>0.07</hackBaseline>
+        <distortionK1>0.0</distortionK1>
+        <distortionK2>0.0</distortionK2>
+        <distortionK3>0.0</distortionK3>
+        <distortionT1>0.0</distortionT1>
+        <distortionT2>0.0</distortionT2>
+      </plugin>
+    </sensor>
+  </gazebo>
 </robot>

File: paul/paul_description/urdf/paul.urdf.xacro (robot description, xacro)
@@ -52,4 +52,5 @@
   <xacro:include filename="$(find paul_description)/urdf/caster.urdf.xacro" />
   <xacro:include filename="$(find paul_description)/urdf/paul.gazebo.xacro" />
+  <xacro:include filename="$(find paul_description)/urdf/lidar.urdf.xacro" />
   <!-- BASE FOOTPRINT -->
   <!-- base_footprint is a fictitious link(frame) that is on the ground right below base_link origin -->
@@ -71,10 +72,11 @@
         <mesh filename="package://paul_description/meshes/shopping-cart-without-wheels.stl"/>
       </geometry>
-      <material name="black"/>
+      <material name="white"/>
     </visual>
     <collision>
       <origin xyz="0.0 0.0 ${base_height/2}" rpy="0.0 0.0 0.0"/>
       <geometry>
-        <box size ="${base_length} ${base_width} ${base_height}" />
+        <!--box size ="${base_length} ${base_width} ${base_height}" /-->
+        <mesh filename="package://paul_description/meshes/shopping-cart-without-wheels.stl"/>
       </geometry>
     </collision>
@@ -92,18 +94,19 @@
     <origin xyz="0 0 0" rpy="0 0 0"/>
   </joint>
-  <!-- LiDAR -->
-  <link name="lidar_link"/>
-  <joint name="baseLidar" type="fixed">
-    <parent link="base_link"/>
-    <child link="lidar_link"/>
-    <origin xyz="0 0 0" rpy="0 0 0"/>
-  </joint>
   <!-- Cameras -->
-  <link name="rgb1_link"/>
+  <link name="rgb1_link" >
+    <visual>
+      <origin xyz="0.0 0.0 0.0" rpy="0.0 0.0 0.0"/>
+      <geometry>
+        <box size ="0.03 0.03 0.03" />
+      </geometry>
+      <material name="black"/>
+    </visual>
+  </link>
   <link name="rgb2_link"/>
   <joint name="baseRGB1" type="fixed">
     <parent link="base_link"/>
     <child link="rgb1_link"/>
-    <origin xyz="0 0 0" rpy="0 0 0"/>
+    <origin xyz="0.592 0.0 0.532" rpy="0 0 0"/>
   </joint>
   <joint name="baseRGB2" type="fixed">
@@ -122,3 +125,7 @@
     <!-- Left caster wheel: "caster_L_link" and "caster_L_joint" -->
   <xacro:caster lr="L" parent="base_link" casterRadius="${wheel_radius}" casterMass="${wheel_mass}" posX="${caster_L_pose_x}" posY="${caster_L_pose_y}" posZ="${caster_L_pose_z}" flipY="1"/>
+  <!-- Lidar sensor -->
+  <xacro:lidar parent="base_link">
+    <origin xyz="0.50614 0 0.1" rpy="0 0 0" />
+  </xacro:lidar>
 </robot>

Commit message: Multi sonar support: - Added sonar to URDF and Gazebo - Modified firmware to use NewPing library

File: paul/paul_description/urdf/paul.gazebo.xacro (robot description, xacro)
@@ -8,4 +8,5 @@
     <turnGravityOff>false</turnGravityOff>
   </gazebo>
+  <!-- wheel controller -->
   <gazebo>
     <plugin name="differential_drive_controller" filename="libgazebo_ros_diff_drive.so">
@@ -30,4 +31,5 @@
     </plugin>
   </gazebo>
+  <!-- rgb camera -->
   <gazebo reference="rgb1_link">
     <sensor type="camera" name="camera1">

File: paul/paul_description/urdf/paul.urdf.xacro (robot description, xacro)
@@ -75,4 +75,5 @@
   <xacro:include filename="$(find paul_description)/urdf/sensors/lidar.urdf.xacro" />
   <xacro:include filename="$(find paul_description)/urdf/sensors/d435/_d435.urdf.xacro"/>
+  <xacro:include filename="$(find paul_description)/urdf/sensors/sonar/sonar.urdf.xacro"/>
   <!-- ============================================== -->
   <!-- ==================== BASE ==================== -->
@@ -159,4 +160,14 @@
     <origin xyz="${realsense_pose_x} ${realsense_pose_y} ${realsense_pose_z}" rpy="${realsense_rot_x} ${realsense_rot_y} ${realsense_rot_z}"/>
   </xacro:sensor_d435>
+  <!-- Sonars -->
+  <xacro:sonar name="left" parent="base_link">
+    <origin xyz="${base_width} 0.1 ${base_height - 0.2}" rpy="0 0 0"/>
+  </xacro:sonar>
+  <xacro:sonar name="center" parent="base_link">
+    <origin xyz="${base_width} 0 ${base_height - 0.2}" rpy="0 0 0"/>
+  </xacro:sonar>
+  <xacro:sonar name="right" parent="base_link">
+    <origin xyz="${base_width} -0.1 ${base_height - 0.2}" rpy="0 0 0"/>
+  </xacro:sonar>
   <!-- ============================================== -->
   <!-- ==================== ARM ===================== -->
