Commit message: Added teleop packages, empty world for gazebo.

File: paul/paul_description/urdf/paul.urdf.xacro (robot description, xacro)
@@ -4,5 +4,5 @@
   <xacro:property name="mass" value="1.0" />
   <!-- Included files -->
-  <xacro:include filename="$(find beam_description)/urdf/Realsense_D455/realsense_d455.urdf.xacro" />
+  <!--xacro:include filename="$(find paul_description)/urdf/Realsense_D455/realsense_d455.urdf.xacro" /-->
   <!-- BASE FOOTPRINT -->
   <!-- base_footprint is a fictitious link(frame) that is on the ground right below base_link origin -->
@@ -28,5 +28,5 @@
       <origin xyz="0.0 0.0 0.0" rpy="1.5708 0.0 3.14159"/>
       <geometry>
-        <mesh filename="package://beam_description/meshes/paul.dae"/>
+        <mesh filename="package://paul_description/meshes/shopping-cart-without-rear-wheels.stl"/>
       </geometry>
       <material name="black"/>
@@ -35,5 +35,5 @@
       <origin xyz="0.0 0.0 0.0" rpy="0.0 0.0 0.0"/>
       <geometry>
-        <mesh filename="package://beam_description/meshes/STL/beam_base.STL" scale="0.001 0.001 0.001"/>
+        <box size ="1.0 1.0 1.0" />
       </geometry>
     </collision>
@@ -42,5 +42,5 @@
     <parent link="base_footprint"/>
     <child link="base_link"/>
-    <origin xyz="0 0 ${Left_wheel_radius - Left_wheel_pose_z}" rpy="0 0 0"/>
+    <origin xyz="0 0 0" rpy="0 0 0"/>
   </joint>
   <!-- IMU -->
@@ -76,9 +76,9 @@
   </joint>
   <!-- Realsense D455 Camera -->
-  <xacro:realsense_d455_sensor parent="head_link" name="realsense" >
+  <!--xacro:realsense_d455_sensor parent="head_link" name="realsense" >
     <origin xyz="${Realsense_pose_x} ${Realsense_pose_y} ${Realsense_pose_z}" rpy="${Realsense_rotation_x} ${Realsense_rotation_y} ${Realsense_rotation_z}"/>
-  </xacro:realsense_d455_sensor>
+  </xacro:realsense_d455_sensor-->
   <!-- Wheels -->
-  <xacro:wheel fb="F" lr="R" parent="base_link" wheelRadius="${Right_wheel_radius}" wheelLength="${Right_wheel_thickness}" wheelMass="${mass/2}" posX="${Right_wheel_pose_x}" posY="${Right_wheel_pose_y}" posZ="${Right_wheel_pose_z}" flipY="1"/>
-  <xacro:wheel fb="F" lr="L" parent="base_link" wheelRadius="${Left_wheel_radius}" wheelLength="${Left_wheel_thickness}" wheelMass="${mass/2}" posX="${Left_wheel_pose_x}" posY="${Left_wheel_pose_y}" posZ="${Left_wheel_pose_z}" flipY="1"/>
+  <!--xacro:wheel fb="F" lr="R" parent="base_link" wheelRadius="${Right_wheel_radius}" wheelLength="${Right_wheel_thickness}" wheelMass="${mass/2}" posX="${Right_wheel_pose_x}" posY="${Right_wheel_pose_y}" posZ="${Right_wheel_pose_z}" flipY="1"/>
+  <xacro:wheel fb="F" lr="L" parent="base_link" wheelRadius="${Left_wheel_radius}" wheelLength="${Left_wheel_thickness}" wheelMass="${mass/2}" posX="${Left_wheel_pose_x}" posY="${Left_wheel_pose_y}" posZ="${Left_wheel_pose_z}" flipY="1"/-->
 </robot>

Commit message: Added rviz config, launch files for simulation, wheel xacro file

File: paul/paul_description/urdf/paul.urdf.xacro (robot description, xacro)
@@ -1,8 +1,31 @@
 <?xml version="1.0"?>
 <robot name="beam" xmlns:xacro="http://www.ros.org/wiki/xacro">
-  <!-- Constant for beam base -->
-  <xacro:property name="mass" value="1.0" />
+  <!-- Constant for paul base -->
+  <xacro:property name="mass" 			value="1.0" />
+  <xacro:property name="base_width" 		value="0.64135" />
+  <xacro:property name="base_height"		value="0.85027" /> <!-- Without wheels -->
+  <xacro:property name="base_length"		value="1.1303" />
+  <xacro:property name="base_pose_z"		value="${base_height/2}" />
+  <!-- Constant for driven wheels -->
+    <!-- Common parameters -->
+  <xacro:property name="Wheel_radius"		value="0.08"/>
+  <xacro:property name="Wheel_thickness"	value="0.055"/>
+  <xacro:property name="Wheel_offset_from_base" value="0.08827" />
+    <!-- Right wheel parameters -->
+  <xacro:property name="Wheel_R_pose_x"		value="0.115"/>
+  <xacro:property name="Wheel_R_pose_y"		value="${- 0.088 - (Right_wheel_thickness/2)}"/>
+  <xacro:property name="Wheel_R_pose_z"		value=" 0.045"/>
+  <xacro:property name="Wheel_R_rot_x"   	value="0.0000"/>
+  <xacro:property name="Wheel_R_rot_y"   	value="1.5707"/>
+  <xacro:property name="Wheel_R_rot_z"   	value="1.5707"/>
+    <!-- Left wheel parameters -->
+  <xacro:property name="Wheel_L_pose_x"		value=" ${Right_wheel_pose_x}"/>
+  <xacro:property name="Wheel_L_pose_y"		value="${-Right_wheel_pose_y}"/>
+  <xacro:property name="Wheel_L_pose_z"		value=" ${Right_wheel_pose_z}"/>
+  <xacro:property name="Wheel_L_rot_x"		value=" ${Right_wheel_rotation_x}"/>
+  <xacro:property name="Wheel_L_rot_y"		value=" ${Rigth_wheel_rotation_y}"/>
+  <xacro:property name="Wheel_L_rot_z"		value=" ${Right_wheel_rotation_z}"/>
   <!-- Included files -->
-  <!--xacro:include filename="$(find paul_description)/urdf/Realsense_D455/realsense_d455.urdf.xacro" /-->
+  <xacro:include filename="$(find paul_description)/urdf/wheel.urdf.xacro" />
   <!-- BASE FOOTPRINT -->
   <!-- base_footprint is a fictitious link(frame) that is on the ground right below base_link origin -->
@@ -26,14 +49,17 @@
     </inertial>
     <visual>
-      <origin xyz="0.0 0.0 0.0" rpy="1.5708 0.0 3.14159"/>
+      <origin xyz="0.0 0.0 ${base_pose_z}" rpy="0.0 0.0 0.0"/>
       <geometry>
+        <box size ="${base_length} ${base_width} ${base_height}" />
+      </geometry>
+      <!--geometry>
         <mesh filename="package://paul_description/meshes/shopping-cart-without-rear-wheels.stl"/>
-      </geometry>
+      </geometry-->
       <material name="black"/>
     </visual>
     <collision>
-      <origin xyz="0.0 0.0 0.0" rpy="0.0 0.0 0.0"/>
+      <origin xyz="0.0 0.0 ${base_height}" rpy="0.0 0.0 0.0"/>
       <geometry>
-        <box size ="1.0 1.0 1.0" />
+        <box size ="${base_length} ${base_width} ${base_height}" />
       </geometry>
     </collision>
@@ -46,9 +72,29 @@
   <!-- IMU -->
   <link name="imu_link"/>
+  <joint name="baseIMU" type="fixed">
+    <parent link="base_link"/>
+    <child link="imu_link"/>
+    <origin xyz="0 0 0" rpy="0 0 0"/>
+  </joint>
   <!-- LiDAR -->
   <link name="lidar_link"/>
+  <joint name="baseLidar" type="fixed">
+    <parent link="base_link"/>
+    <child link="lidar_link"/>
+    <origin xyz="0 0 0" rpy="0 0 0"/>
+  </joint>
   <!-- Cameras -->
   <link name="rgb1_link"/>
   <link name="rgb2_link"/>
+  <joint name="baseRGB1" type="fixed">
+    <parent link="base_link"/>
+    <child link="rgb1_link"/>
+    <origin xyz="0 0 0" rpy="0 0 0"/>
+  </joint>
+  <joint name="baseRGB2" type="fixed">
+    <parent link="base_link"/>
+    <child link="rgb2_link"/>
+    <origin xyz="0 0 0" rpy="0 0 0"/>
+  </joint>
   <!-- Robot arm -->
   <link name="arm_j1_link"/>
@@ -60,15 +106,10 @@
     <origin xyz="0 0 0" rpy="0 0 0"/>
   </joint>
-  <joint name="arm_j1_j2" type="revolute">
+  <joint name="arm_j1_j2" type="fixed">
     <parent link="arm_j1_link"/>
     <child link="arm_j2_link"/>
     <origin xyz="0 0 0" rpy="0 0 0"/>
   </joint>
-  <joint name="arm_j1_j2" type="revolute">
-    <parent link="arm_j1_link"/>
-    <child link="arm_j2_link"/>
-    <origin xyz="0 0 0" rpy="0 0 0"/>
-  </joint>
-  <joint name="arm_j2_j3" type="prismatic">
+  <joint name="arm_j2_j3" type="fixed">
     <parent link="arm_j2_link"/>
     <child link="arm_j3_link"/>
@@ -79,6 +120,6 @@
     <origin xyz="${Realsense_pose_x} ${Realsense_pose_y} ${Realsense_pose_z}" rpy="${Realsense_rotation_x} ${Realsense_rotation_y} ${Realsense_rotation_z}"/>
   </xacro:realsense_d455_sensor-->
-  <!-- Wheels -->
-  <!--xacro:wheel fb="F" lr="R" parent="base_link" wheelRadius="${Right_wheel_radius}" wheelLength="${Right_wheel_thickness}" wheelMass="${mass/2}" posX="${Right_wheel_pose_x}" posY="${Right_wheel_pose_y}" posZ="${Right_wheel_pose_z}" flipY="1"/>
+  <!-- Wheels --><!--
+  <xacro:wheel fb="F" lr="R" parent="base_link" wheelRadius="${Right_wheel_radius}" wheelLength="${Right_wheel_thickness}" wheelMass="${mass/2}" posX="${Right_wheel_pose_x}" posY="${Right_wheel_pose_y}" posZ="${Right_wheel_pose_z}" flipY="1"/>
   <xacro:wheel fb="F" lr="L" parent="base_link" wheelRadius="${Left_wheel_radius}" wheelLength="${Left_wheel_thickness}" wheelMass="${mass/2}" posX="${Left_wheel_pose_x}" posY="${Left_wheel_pose_y}" posZ="${Left_wheel_pose_z}" flipY="1"/-->
 </robot>

Commit message: Modified robot description to fit new CAD, support for mesh added.

File: paul/paul_description/urdf/paul.urdf.xacro (robot description, xacro)
@@ -6,54 +6,47 @@
   <xacro:property name="base_height"		value="0.85027" /> <!-- Without wheels -->
   <xacro:property name="base_length"		value="1.1303" />
-  <xacro:property name="base_pose_z"		value="${base_height/2}" />
+  <xacro:property name="base_pose_z"		value="${ground_to_base_z}" />
+  <xacro:property name="wheel_to_base_z" 	value="0.08827" />
+  <xacro:property name="ground_to_base_z"	value="${wheel_to_base_z + wheel_radius}" />
   <!-- Constant for driven wheels -->
     <!-- Common parameters -->
-  <xacro:property name="Wheel_radius"		value="0.08"/>
-  <xacro:property name="Wheel_thickness"	value="0.055"/>
-  <xacro:property name="Wheel_offset_from_base" value="0.08827" />
+  <xacro:property name="wheel_diameter"		value="0.14732" />
+  <xacro:property name="wheel_radius"		value="${wheel_diameter/2}"/>
+  <xacro:property name="wheel_thickness"	value="0.055"/>
+  <xacro:property name="front_to_rear_wheels_x"	value="0.84056"/>
+  <xacro:property name="front_right_left_y"	value="0.3302"/>
+  <xacro:property name="rear_right_left_y"	value="0.5715"/>
     <!-- Right wheel parameters -->
-  <xacro:property name="Wheel_R_pose_x"		value="0.115"/>
-  <xacro:property name="Wheel_R_pose_y"		value="${- 0.088 - (Right_wheel_thickness/2)}"/>
-  <xacro:property name="Wheel_R_pose_z"		value=" 0.045"/>
-  <xacro:property name="Wheel_R_rot_x"   	value="0.0000"/>
-  <xacro:property name="Wheel_R_rot_y"   	value="1.5707"/>
-  <xacro:property name="Wheel_R_rot_z"   	value="1.5707"/>
+  <xacro:property name="wheel_R_pose_x"		value="${-front_to_rear_wheels_x/2}"/>
+  <xacro:property name="wheel_R_pose_y"		value="${-rear_right_left_y/2}"/>
+  <xacro:property name="wheel_R_pose_z"		value="${-wheel_radius}"/>
+  <xacro:property name="wheel_R_rot_x"   	value="0.0000"/>
+  <xacro:property name="wheel_R_rot_y"   	value="0.0000"/>
+  <xacro:property name="wheel_R_rot_z"   	value="0.0000"/>
     <!-- Left wheel parameters -->
-  <xacro:property name="Wheel_L_pose_x"		value=" ${Right_wheel_pose_x}"/>
-  <xacro:property name="Wheel_L_pose_y"		value="${-Right_wheel_pose_y}"/>
-  <xacro:property name="Wheel_L_pose_z"		value=" ${Right_wheel_pose_z}"/>
-  <xacro:property name="Wheel_L_rot_x"		value=" ${Right_wheel_rotation_x}"/>
-  <xacro:property name="Wheel_L_rot_y"		value=" ${Rigth_wheel_rotation_y}"/>
-  <xacro:property name="Wheel_L_rot_z"		value=" ${Right_wheel_rotation_z}"/>
+  <xacro:property name="wheel_L_pose_x"		value=" ${wheel_R_pose_x}"/>
+  <xacro:property name="wheel_L_pose_y"		value="${-wheel_R_pose_y}"/>
+  <xacro:property name="wheel_L_pose_z"		value=" ${wheel_R_pose_z}"/>
+  <xacro:property name="wheel_L_rot_x"		value=" ${wheel_R_rot_x}"/>
+  <xacro:property name="wheel_L_rot_y"		value=" ${wheel_R_rot_y}"/>
+  <xacro:property name="wheel_L_rot_z"		value=" ${wheel_R_rot_z}"/>
   <!-- Included files -->
   <xacro:include filename="$(find paul_description)/urdf/wheel.urdf.xacro" />
   <!-- BASE FOOTPRINT -->
   <!-- base_footprint is a fictitious link(frame) that is on the ground right below base_link origin -->
-  <link name="base_footprint">
-    <visual>
-      <origin xyz="0 0 0" rpy="0 0 0" />
-      <geometry>
-        <box size ="0.001 0.001 0.001" />
-      </geometry>
-    </visual>
-  </link>
+  <link name="base_footprint"/>
   <!-- BASE_LINK (only static pieces) -->
   <link name="base_link">
     <inertial>
-      <origin xyz="0.01336 0.0 0.07595" rpy="0.0 0.0 0.0"/>
-      <mass value="9.0"/>
-      <inertia
-        ixx="0" ixy="0" ixz="0"
-        iyy="0" iyz="0"
-        izz="0" />
+      <mass value="1" />
+      <inertia  ixx="0.001" ixy="0.0"  ixz="0.0"
+                iyy="0.001"  iyz="0.0"
+                izz="0.001" />
     </inertial>
     <visual>
-      <origin xyz="0.0 0.0 ${base_pose_z}" rpy="0.0 0.0 0.0"/>
+      <origin xyz="0.0 0.0 ${-ground_to_base_z}" rpy="0.0 0.0 0.0"/>
       <geometry>
-        <box size ="${base_length} ${base_width} ${base_height}" />
+        <mesh filename="package://paul_description/meshes/shopping-cart-without-wheels.stl"/>
       </geometry>
-      <!--geometry>
-        <mesh filename="package://paul_description/meshes/shopping-cart-without-rear-wheels.stl"/>
-      </geometry-->
       <material name="black"/>
     </visual>
@@ -68,5 +61,5 @@
     <parent link="base_footprint"/>
     <child link="base_link"/>
-    <origin xyz="0 0 0" rpy="0 0 0"/>
+    <origin xyz="0.0 0.0 ${ground_to_base_z}" rpy="0 0 0"/>
   </joint>
   <!-- IMU -->
@@ -120,5 +113,5 @@
     <origin xyz="${Realsense_pose_x} ${Realsense_pose_y} ${Realsense_pose_z}" rpy="${Realsense_rotation_x} ${Realsense_rotation_y} ${Realsense_rotation_z}"/>
   </xacro:realsense_d455_sensor-->
-  <!-- Wheels --><!--
+  <!-- wheels --><!--
   <xacro:wheel fb="F" lr="R" parent="base_link" wheelRadius="${Right_wheel_radius}" wheelLength="${Right_wheel_thickness}" wheelMass="${mass/2}" posX="${Right_wheel_pose_x}" posY="${Right_wheel_pose_y}" posZ="${Right_wheel_pose_z}" flipY="1"/>
   <xacro:wheel fb="F" lr="L" parent="base_link" wheelRadius="${Left_wheel_radius}" wheelLength="${Left_wheel_thickness}" wheelMass="${mass/2}" posX="${Left_wheel_pose_x}" posY="${Left_wheel_pose_y}" posZ="${Left_wheel_pose_z}" flipY="1"/-->

Commit message: Working differential drive with caster wheels.

File: paul/paul_description/urdf/paul.urdf.xacro (robot description, xacro)
@@ -2,5 +2,5 @@
 <robot name="beam" xmlns:xacro="http://www.ros.org/wiki/xacro">
   <!-- Constant for paul base -->
-  <xacro:property name="mass" 			value="1.0" />
+  <xacro:property name="mass" 			value="20.0" />
   <xacro:property name="base_width" 		value="0.64135" />
   <xacro:property name="base_height"		value="0.85027" /> <!-- Without wheels -->
@@ -9,12 +9,13 @@
   <xacro:property name="wheel_to_base_z" 	value="0.08827" />
   <xacro:property name="ground_to_base_z"	value="${wheel_to_base_z + wheel_radius}" />
-  <!-- Constant for driven wheels -->
-    <!-- Common parameters -->
+  <!-- Common wheels parameters -->
   <xacro:property name="wheel_diameter"		value="0.14732" />
   <xacro:property name="wheel_radius"		value="${wheel_diameter/2}"/>
-  <xacro:property name="wheel_thickness"	value="0.055"/>
+  <xacro:property name="wheel_thickness"	value="0.03"/>
+  <xacro:property name="wheel_mass"		value="0.200"/>
   <xacro:property name="front_to_rear_wheels_x"	value="0.84056"/>
   <xacro:property name="front_right_left_y"	value="0.3302"/>
   <xacro:property name="rear_right_left_y"	value="0.5715"/>
+  <!-- Constant for driven wheels -->
     <!-- Right wheel parameters -->
   <xacro:property name="wheel_R_pose_x"		value="${-front_to_rear_wheels_x/2}"/>
@@ -31,6 +32,24 @@
   <xacro:property name="wheel_L_rot_y"		value=" ${wheel_R_rot_y}"/>
   <xacro:property name="wheel_L_rot_z"		value=" ${wheel_R_rot_z}"/>
+  <!-- Constant for caster wheels -->
+    <!-- Right caster wheel parameters -->
+  <xacro:property name="caster_R_pose_x"	value="${front_to_rear_wheels_x/2}"/>
+  <xacro:property name="caster_R_pose_y"	value="${-front_right_left_y/2}"/>
+  <xacro:property name="caster_R_pose_z"	value="${-wheel_radius}"/>
+  <xacro:property name="caster_R_rot_x"   	value="0.0000"/>
+  <xacro:property name="caster_R_rot_y"   	value="0.0000"/>
+  <xacro:property name="caster_R_rot_z"   	value="0.0000"/>
+    <!-- Left caster wheel parameters -->
+  <xacro:property name="caster_L_pose_x"	value=" ${caster_R_pose_x}"/>
+  <xacro:property name="caster_L_pose_y"	value="${-caster_R_pose_y}"/>
+  <xacro:property name="caster_L_pose_z"	value=" ${caster_R_pose_z}"/>
+  <xacro:property name="caster_L_rot_x"		value=" ${caster_R_rot_x}"/>
+  <xacro:property name="caster_L_rot_y"		value=" ${caster_R_rot_y}"/>
+  <xacro:property name="caster_L_rot_z"		value=" ${caster_R_rot_z}"/>
+    <!-- Left caster wheel parameters -->
   <!-- Included files -->
   <xacro:include filename="$(find paul_description)/urdf/wheel.urdf.xacro" />
+  <xacro:include filename="$(find paul_description)/urdf/caster.urdf.xacro" />
+  <xacro:include filename="$(find paul_description)/urdf/paul.gazebo.xacro" />
   <!-- BASE FOOTPRINT -->
   <!-- base_footprint is a fictitious link(frame) that is on the ground right below base_link origin -->
@@ -90,29 +109,13 @@
     <origin xyz="0 0 0" rpy="0 0 0"/>
   </joint>
-  <!-- Robot arm -->
-  <link name="arm_j1_link"/>
-  <link name="arm_j2_link"/>
-  <link name="arm_j3_link"/>
-  <joint name="baseArm_j1" type="fixed">
-    <parent link="base_link"/>
-    <child link="arm_j1_link"/>
-    <origin xyz="0 0 0" rpy="0 0 0"/>
-  </joint>
-  <joint name="arm_j1_j2" type="fixed">
-    <parent link="arm_j1_link"/>
-    <child link="arm_j2_link"/>
-    <origin xyz="0 0 0" rpy="0 0 0"/>
-  </joint>
-  <joint name="arm_j2_j3" type="fixed">
-    <parent link="arm_j2_link"/>
-    <child link="arm_j3_link"/>
-    <origin xyz="0 0 0" rpy="0 0 0"/>
-  </joint>
-  <!-- Realsense D455 Camera -->
-  <!--xacro:realsense_d455_sensor parent="head_link" name="realsense" >
-    <origin xyz="${Realsense_pose_x} ${Realsense_pose_y} ${Realsense_pose_z}" rpy="${Realsense_rotation_x} ${Realsense_rotation_y} ${Realsense_rotation_z}"/>
-  </xacro:realsense_d455_sensor-->
-  <!-- wheels --><!--
-  <xacro:wheel fb="F" lr="R" parent="base_link" wheelRadius="${Right_wheel_radius}" wheelLength="${Right_wheel_thickness}" wheelMass="${mass/2}" posX="${Right_wheel_pose_x}" posY="${Right_wheel_pose_y}" posZ="${Right_wheel_pose_z}" flipY="1"/>
-  <xacro:wheel fb="F" lr="L" parent="base_link" wheelRadius="${Left_wheel_radius}" wheelLength="${Left_wheel_thickness}" wheelMass="${mass/2}" posX="${Left_wheel_pose_x}" posY="${Left_wheel_pose_y}" posZ="${Left_wheel_pose_z}" flipY="1"/-->
+  <!-- driven wheels -->
+    <!-- Right Wheel: "wheel_R_link" and "wheel_R_joint" -->
+  <xacro:wheel lr="R" parent="base_link" wheelRadius="${wheel_radius}" wheelLength="${wheel_thickness}" wheelMass="${wheel_mass}" posX="${wheel_R_pose_x}" posY="${wheel_R_pose_y}" posZ="${wheel_R_pose_z}" flipY="1"/>
+    <!-- Left Wheel: "wheel_L_link" and "wheel_L_joint" -->
+  <xacro:wheel lr="L" parent="base_link" wheelRadius="${wheel_radius}" wheelLength="${wheel_thickness}" wheelMass="${wheel_mass}" posX="${wheel_L_pose_x}" posY="${wheel_L_pose_y}" posZ="${wheel_L_pose_z}" flipY="1"/>
+  <!-- caster wheels -->
+    <!-- Right caster wheel: "caster_R_link" and "caster_R_joint" -->
+  <xacro:caster lr="R" parent="base_link" casterRadius="${wheel_radius}" casterMass="${wheel_mass}" posX="${caster_R_pose_x}" posY="${caster_R_pose_y}" posZ="${caster_R_pose_z}" flipY="1"/>
+    <!-- Left caster wheel: "caster_L_link" and "caster_L_joint" -->
+  <xacro:caster lr="L" parent="base_link" casterRadius="${wheel_radius}" casterMass="${wheel_mass}" posX="${caster_L_pose_x}" posY="${caster_L_pose_y}" posZ="${caster_L_pose_z}" flipY="1"/>
 </robot>

File: paul/paul_description/urdf/wheel.urdf.xacro (robot description, xacro)
@@ -9,7 +9,7 @@
               izz="${m*r*r/2}" />
   </xacro:macro>
-  <!--fb : Front/Back => F/B ; lr: Left/Right => L/R -->
-  <xacro:macro name="wheel" params="fb lr parent wheelRadius wheelLength wheelMass posX posY posZ flipY">
-    <link name="wheel${fb}${lr}_link">
+  <!-- lr: Left/Right => L/R -->
+  <xacro:macro name="wheel" params="lr parent wheelRadius wheelLength wheelMass posX posY posZ flipY">
+    <link name="wheel_${lr}_link">
       <visual>
         <origin xyz="0 0 0" rpy="${flipY*PI/2} 0  0 " />
@@ -44,5 +44,5 @@
       </inertial>
     </link>
-    <gazebo reference="wheel${fb}${lr}_link">
+    <gazebo reference="wheel_${lr}_link">
       <mu1 value="1.0"/>
       <mu2 value="1.0"/>
@@ -53,7 +53,7 @@
       <turnGravityOff>false</turnGravityOff>
     </gazebo>
-    <joint name="wheel${fb}${lr}_joint" type="continuous">
+    <joint name="wheel_${lr}_joint" type="continuous">
       <parent link="${parent}"/>
-      <child link="wheel${fb}${lr}_link"/>
+      <child link="wheel_${lr}_link"/>
       <origin xyz="${posX} ${posY} ${posZ}" rpy="0 0 0" />
       <axis xyz="0 1 0" rpy="0  0" />
@@ -62,8 +62,8 @@
     </joint>
     <!-- Transmission is important to link the joints and the controller -->
-    <transmission name="$wheel${fb}${lr}_joint_trans">
+    <transmission name="$wheel_${lr}_joint_trans">
       <type>transmission_interface/SimpleTransmission</type>
-      <joint name="$wheel${fb}${lr}_joint" />
-      <actuator name="$wheel${fb}${lr}_joint_motor">
+      <joint name="$wheel_${lr}_joint" />
+      <actuator name="$wheel_${lr}_joint_motor">
         <hardwareInterface>EffortJointInterface</hardwareInterface>
         <mechanicalReduction>1</mechanicalReduction>

Commit message: Model working in gazebo

File: paul/paul_description/urdf/paul.urdf.xacro (robot description, xacro)
@@ -58,11 +58,14 @@
   <link name="base_link">
     <inertial>
-      <mass value="1" />
-      <inertia  ixx="0.001" ixy="0.0"  ixz="0.0"
-                iyy="0.001"  iyz="0.0"
-                izz="0.001" />
+      <mass value="24.265" />
+      <!-- Position of center of mass -->
+      <origin xyz="-0.176 0.0 0.203" rpy="0 0 0" />
+      <!-- Moment of inertia around center of mass -->
+      <inertia  ixx="3.681" ixy="0.0"  ixz="-0.168"
+                iyy="4.665"  iyz="0.0"
+                izz="3.867" />
     </inertial>
     <visual>
-      <origin xyz="0.0 0.0 ${-ground_to_base_z}" rpy="0.0 0.0 0.0"/>
+      <origin xyz="0.0 0.0 0.0" rpy="0.0 0.0 0.0"/>
       <geometry>
         <mesh filename="package://paul_description/meshes/shopping-cart-without-wheels.stl"/>
@@ -71,5 +74,5 @@
     </visual>
     <collision>
-      <origin xyz="0.0 0.0 ${base_height}" rpy="0.0 0.0 0.0"/>
+      <origin xyz="0.0 0.0 ${base_height/2}" rpy="0.0 0.0 0.0"/>
       <geometry>
         <box size ="${base_length} ${base_width} ${base_height}" />
