Commit message: Added move_base, RGB-D Camera support (realsense)

File: paul/paul_description/urdf/paul.urdf.xacro (robot description, xacro)
@@ -1,4 +1,4 @@
 <?xml version="1.0"?>
-<robot name="beam" xmlns:xacro="http://www.ros.org/wiki/xacro">
+<robot name="paul" xmlns:xacro="http://www.ros.org/wiki/xacro">
   <!-- Constant for paul base -->
   <xacro:property name="mass" 			value="20.0" />
@@ -47,5 +47,11 @@
   <xacro:property name="caster_L_rot_y"		value=" ${caster_R_rot_y}"/>
   <xacro:property name="caster_L_rot_z"		value=" ${caster_R_rot_z}"/>
-    <!-- Left caster wheel parameters -->
+  <!-- RGBD Sensor parameters -->
+  <xacro:property name="realsense_pose_x" value="${base_width/2}" />
+  <xacro:property name="realsense_pose_y" value="0.0" />
+  <xacro:property name="realsense_pose_z" value="${base_height}" />
+  <xacro:property name="realsense_rot_x" value="0.0" />
+  <xacro:property name="realsense_rot_y" value="0.0" />
+  <xacro:property name="realsense_rot_z" value="0.0" />
   <!-- Included files -->
   <xacro:include filename="$(find paul_description)/urdf/wheel.urdf.xacro" />
@@ -53,4 +59,5 @@
   <xacro:include filename="$(find paul_description)/urdf/paul.gazebo.xacro" />
   <xacro:include filename="$(find paul_description)/urdf/lidar.urdf.xacro" />
+  <xacro:include filename="$(find paul_description)/urdf/realsense_d415.urdf.xacro"/>
   <!-- BASE FOOTPRINT -->
   <!-- base_footprint is a fictitious link(frame) that is on the ground right below base_link origin -->
@@ -129,3 +136,7 @@
     <origin xyz="0.50614 0 0.1" rpy="0 0 0" />
   </xacro:lidar>
+  <!-- RGB-D Sensor -->
+  <xacro:realsense_d415_sensor parent="base_link" name="rgbd_realsense" >
+    <origin xyz="${realsense_pose_x} ${realsense_pose_y} ${realsense_pose_z}" rpy="${realsense_rot_x} ${realsense_rot_y} ${realsense_rot_z}"/>
+  </xacro:realsense_d415_sensor>
 </robot>

Commit message: Navigation working (tuning needed)

File: paul/paul_description/urdf/paul.urdf.xacro (robot description, xacro)
@@ -48,5 +48,5 @@
   <xacro:property name="caster_L_rot_z"		value=" ${caster_R_rot_z}"/>
   <!-- RGBD Sensor parameters -->
-  <xacro:property name="realsense_pose_x" value="${base_width/2}" />
+  <xacro:property name="realsense_pose_x" value="${base_width}" />
   <xacro:property name="realsense_pose_y" value="0.0" />
   <xacro:property name="realsense_pose_z" value="${base_height}" />
@@ -137,5 +137,5 @@
   </xacro:lidar>
   <!-- RGB-D Sensor -->
-  <xacro:realsense_d415_sensor parent="base_link" name="rgbd_realsense" >
+  <xacro:realsense_d415_sensor parent="base_link" name="realsense" >
     <origin xyz="${realsense_pose_x} ${realsense_pose_y} ${realsense_pose_z}" rpy="${realsense_rot_x} ${realsense_rot_y} ${realsense_rot_z}"/>
   </xacro:realsense_d415_sensor>

Commit message: Refactoring et intégration de la D435: - Début documentation dans le README - Ajout de la D435 au URDF, à la simulation et dans le launch file - Ajout des dépendances pour les différents packages - Refactoring avec l'ajout de launch file pour simplifier le bringup

File: paul/paul_description/urdf/paul.urdf.xacro (robot description, xacro)
@@ -1,4 +1,9 @@
 <?xml version="1.0"?>
 <robot name="paul" xmlns:xacro="http://www.ros.org/wiki/xacro">
+  <!-- Need argument to get from launch file:
+  based on https://answers.ros.org/question/379014/passing-outside-parameters-into-urdf-file-using-xacro/ -->
+  <xacro:arg name="simulation" default="true"/>
+  <!-- Need seperate property for xacro inorder processing -->
+  <xacro:property name="simulation" value="$(arg simulation)"/>
   <!-- Constant for paul base -->
   <xacro:property name="mass" 			value="20.0" />
@@ -59,5 +64,5 @@
   <xacro:include filename="$(find paul_description)/urdf/paul.gazebo.xacro" />
   <xacro:include filename="$(find paul_description)/urdf/lidar.urdf.xacro" />
-  <xacro:include filename="$(find paul_description)/urdf/realsense_d415.urdf.xacro"/>
+  <xacro:include filename="$(find paul_description)/urdf/d435/_d435.urdf.xacro"/>
   <!-- BASE FOOTPRINT -->
   <!-- base_footprint is a fictitious link(frame) that is on the ground right below base_link origin -->
@@ -136,7 +141,7 @@
     <origin xyz="0.50614 0 0.1" rpy="0 0 0" />
   </xacro:lidar>
-  <!-- RGB-D Sensor -->
-  <xacro:realsense_d415_sensor parent="base_link" name="realsense" >
+  <!-- D435 RGB-D Sensor -->
+  <xacro:sensor_d435 parent="base_link" use_nominal_extrinsics="${simulation}">
     <origin xyz="${realsense_pose_x} ${realsense_pose_y} ${realsense_pose_z}" rpy="${realsense_rot_x} ${realsense_rot_y} ${realsense_rot_z}"/>
-  </xacro:realsense_d415_sensor>
+  </xacro:sensor_d435>
 </robot>

Commit message: Added kinova arm in robot model

File: paul/paul_description/urdf/paul.urdf.xacro (robot description, xacro)
@@ -60,8 +60,9 @@
   <xacro:property name="realsense_rot_z" value="0.0" />
   <!-- Included files -->
-  <xacro:include filename="$(find paul_description)/urdf/wheel.urdf.xacro" />
-  <xacro:include filename="$(find paul_description)/urdf/caster.urdf.xacro" />
+  <xacro:include filename="$(find paul_description)/urdf/components/wheel.urdf.xacro" />
+  <xacro:include filename="$(find paul_description)/urdf/components/caster.urdf.xacro" />
   <xacro:include filename="$(find paul_description)/urdf/paul.gazebo.xacro" />
-  <xacro:include filename="$(find paul_description)/urdf/lidar.urdf.xacro" />
+  <xacro:include filename="$(find paul_description)/urdf/sensors/lidar.urdf.xacro" />
+  <xacro:include filename="$(find paul_description)/urdf/arms/gen3_lite.urdf.xacro" />
   <xacro:include filename="$(find paul_description)/urdf/d435/_d435.urdf.xacro"/>
   <!-- BASE FOOTPRINT -->
@@ -127,4 +128,10 @@
     <origin xyz="0 0 0" rpy="0 0 0"/>
   </joint>
+  <!-- Arm -->
+  <joint name="baseArm" type="fixed">
+    <parent link="base_link"/>
+    <child link="gen3_lite_base_link"/>
+    <origin xyz="-0.6 0.0 0.5" rpy="0 0 0"/>
+  </joint>
   <!-- driven wheels -->
     <!-- Right Wheel: "wheel_R_link" and "wheel_R_joint" -->

Commit message: added linear axis in model and joint gui for visualizing

File: paul/paul_description/urdf/paul.urdf.xacro (robot description, xacro)
@@ -128,9 +128,17 @@
     <origin xyz="0 0 0" rpy="0 0 0"/>
   </joint>
+  <!-- Arm linear axis -->
+  <link name="linearAxis_link" />
+  <joint name="linearAxis" type="prismatic">
+    <limit effort="1000.0" lower="0" upper="1" velocity="0.5"/>
+    <parent link="base_link"/>
+    <child link="linearAxis_link"/>
+    <origin xyz="-0.6 0.0 0.0" rpy="0 -1.5708 0"/>
+  </joint>
   <!-- Arm -->
   <joint name="baseArm" type="fixed">
-    <parent link="base_link"/>
+    <parent link="linearAxis_link"/>
     <child link="gen3_lite_base_link"/>
-    <origin xyz="-0.6 0.0 0.5" rpy="0 0 0"/>
+    <origin xyz="0.0 0.0 0.0" rpy="0 1.5708 0"/>
   </joint>
   <!-- driven wheels -->

Commit message: Grocery layout: - Modified shelves with simple shapes (boxes) - 8x_... are now a single model - Added world.launch for easier debugging - Added testbench.world, but not ready - Added logo model, still need to do UV projection on cylinder - Modified URDF model, since branch created from wrong commit

File: paul/paul_description/urdf/paul.urdf.xacro (robot description, xacro)
@@ -64,5 +64,4 @@
   <xacro:include filename="$(find paul_description)/urdf/paul.gazebo.xacro" />
   <xacro:include filename="$(find paul_description)/urdf/sensors/lidar.urdf.xacro" />
-  <xacro:include filename="$(find paul_description)/urdf/arms/gen3_lite.urdf.xacro" />
   <xacro:include filename="$(find paul_description)/urdf/d435/_d435.urdf.xacro"/>
   <!-- BASE FOOTPRINT -->
@@ -128,10 +127,4 @@
     <origin xyz="0 0 0" rpy="0 0 0"/>
   </joint>
-  <!-- Arm -->
-  <joint name="baseArm" type="fixed">
-    <parent link="base_link"/>
-    <child link="gen3_lite_base_link"/>
-    <origin xyz="-0.6 0.0 0.5" rpy="0 0 0"/>
-  </joint>
   <!-- driven wheels -->
     <!-- Right Wheel: "wheel_R_link" and "wheel_R_joint" -->

Commit message: Fixed URDF arm inclusion for simulation

File: paul/paul_description/urdf/paul.urdf.xacro (robot description, xacro)
@@ -3,10 +3,10 @@
   <!-- Need argument to get from launch file:
   based on https://answers.ros.org/question/379014/passing-outside-parameters-into-urdf-file-using-xacro/ -->
-  <xacro:arg name="simulation" default="true"/>
+  <xacro:arg name="sim" default="true"/>
   <!-- Kinova arm parameters -->
   <xacro:arg name="arm"        default="gen3_lite"/>
   <xacro:arg name="gripper"    default="gen3_lite_2f"/>
   <!-- Need seperate property for xacro inorder processing -->
-  <xacro:property name="simulation" value="$(arg simulation)"/>
+  <xacro:property name="sim" value="$(arg sim)"/>
   <!-- Constant for paul base -->
   <xacro:property name="mass" 			value="20.0" />
@@ -67,5 +67,4 @@
   <xacro:include filename="$(find paul_description)/urdf/paul.gazebo.xacro" />
   <xacro:include filename="$(find paul_description)/urdf/sensors/lidar.urdf.xacro" />
-  <xacro:include filename="$(find paul_description)/urdf/arms/$(arg arm)_$(arg gripper).xacro"/>
   <xacro:include filename="$(find paul_description)/urdf/d435/_d435.urdf.xacro"/>
   <!-- BASE FOOTPRINT -->
@@ -139,5 +138,5 @@
     <origin xyz="-0.6 0.0 0.0" rpy="0 -1.5708 0"/>
   </joint>
-  <!-- Arm -->
+  <!-- Arm: xacro must be after so the baseArm joint exists -->
   <joint name="baseArm" type="fixed">
     <parent link="linearAxis_link"/>
@@ -145,4 +144,5 @@
     <origin xyz="0.0 0.0 0.0" rpy="0 1.5708 0"/>
   </joint>
+  <xacro:include filename="$(find paul_description)/urdf/arms/arm.xacro"/>
   <!-- driven wheels -->
     <!-- Right Wheel: "wheel_R_link" and "wheel_R_joint" -->
@@ -160,5 +160,5 @@
   </xacro:lidar>
   <!-- D435 RGB-D Sensor -->
-  <xacro:sensor_d435 parent="base_link" use_nominal_extrinsics="${simulation}">
+  <xacro:sensor_d435 parent="base_link" use_nominal_extrinsics="${sim}">
     <origin xyz="${realsense_pose_x} ${realsense_pose_y} ${realsense_pose_z}" rpy="${realsense_rot_x} ${realsense_rot_y} ${realsense_rot_z}"/>
   </xacro:sensor_d435>

Commit message: README conflict resolution

File: paul/paul_description/urdf/paul.urdf.xacro (robot description, xacro)
@@ -3,10 +3,10 @@
   <!-- Need argument to get from launch file:
   based on https://answers.ros.org/question/379014/passing-outside-parameters-into-urdf-file-using-xacro/ -->
-  <xacro:arg name="simulation" default="true"/>
-  <!-- Kinova arm parameters -->
-  <xacro:arg name="arm"        default="gen3_lite"/>
-  <xacro:arg name="gripper"    default="gen3_lite_2f"/>
-  <!-- Need seperate property for xacro inorder processing -->
-  <xacro:property name="simulation" value="$(arg simulation)"/>
+  <xacro:arg name="arm"     default="$(optenv PAUL_ARM_MODEL gen3_lite)" />
+  <xacro:arg name="dof"     default="$(optenv PAUL_ARM_DOF 6)" />
+  <xacro:arg name="vision"  default="$(optenv PAUL_ARM_VISION false)" />
+  <xacro:arg name="gripper" default="$(optenv PAUL_ARM_GRIPPER gen3_lite_2f)" />
+  <xacro:arg name="sim"     default="$(optenv PAUL_ARM_SIM false)" />
+  <xacro:arg name="prefix"  default="$(optenv PAUL_ARM_PREFIX arm_)" />
   <!-- Constant for paul base -->
   <xacro:property name="mass" 			value="20.0" />
@@ -59,4 +59,5 @@
   <xacro:property name="realsense_pose_y" value="0.0" />
   <xacro:property name="realsense_pose_z" value="${base_height}" />
+  <xacro:property name="use_nominal_extrinsics" value="$(arg sim)"/>
   <xacro:property name="realsense_rot_x" value="0.0" />
   <xacro:property name="realsense_rot_y" value="0.0" />
@@ -67,6 +68,6 @@
   <xacro:include filename="$(find paul_description)/urdf/paul.gazebo.xacro" />
   <xacro:include filename="$(find paul_description)/urdf/sensors/lidar.urdf.xacro" />
-  <xacro:include filename="$(find paul_description)/urdf/arms/$(arg arm)_$(arg gripper).xacro"/>
   <xacro:include filename="$(find paul_description)/urdf/d435/_d435.urdf.xacro"/>
+  <xacro:include filename="$(find paul_description)/urdf/arms/paul_gen3_lite_description.urdf.xacro" />
   <!-- BASE FOOTPRINT -->
   <!-- base_footprint is a fictitious link(frame) that is on the ground right below base_link origin -->
@@ -91,7 +92,6 @@
     </visual>
     <collision>
-      <origin xyz="0.0 0.0 ${base_height/2}" rpy="0.0 0.0 0.0"/>
+      <origin xyz="0.0 0.0 0.0" rpy="0.0 0.0 0.0"/>
       <geometry>
-        <!--box size ="${base_length} ${base_width} ${base_height}" /-->
         <mesh filename="package://paul_description/meshes/shopping-cart-without-wheels.stl"/>
       </geometry>
@@ -139,9 +139,9 @@
     <origin xyz="-0.6 0.0 0.0" rpy="0 -1.5708 0"/>
   </joint>
-  <!-- Arm -->
-  <joint name="baseArm" type="fixed">
+  <link name="armMount_link"/>
+  <joint name="armMount" type="fixed">
     <parent link="linearAxis_link"/>
-    <child link="$(arg arm)_$(arg gripper)_base_link"/>
-    <origin xyz="0.0 0.0 0.0" rpy="0 1.5708 0"/>
+    <child link="armMount_link"/>
+    <origin xyz="0.0 0.0 0.0" rpy="0.0 0.0 0.0"/>
   </joint>
   <!-- driven wheels -->
@@ -160,5 +160,5 @@
   </xacro:lidar>
   <!-- D435 RGB-D Sensor -->
-  <xacro:sensor_d435 parent="base_link" use_nominal_extrinsics="${simulation}">
+  <xacro:sensor_d435 parent="base_link" use_nominal_extrinsics="${use_nominal_extrinsics}">
     <origin xyz="${realsense_pose_x} ${realsense_pose_y} ${realsense_pose_z}" rpy="${realsense_rot_x} ${realsense_rot_y} ${realsense_rot_z}"/>
   </xacro:sensor_d435>

Commit message: Testbench and grocery worlds improvements: - Added raise displays in grocery - Finished testbench and created a simplified version - Added SDF models of food

File: paul/paul_description/urdf/paul.urdf.xacro (robot description, xacro)
@@ -92,6 +92,6 @@
       <origin xyz="0.0 0.0 ${base_height/2}" rpy="0.0 0.0 0.0"/>
       <geometry>
-        <!--box size ="${base_length} ${base_width} ${base_height}" /-->
-        <mesh filename="package://paul_description/meshes/shopping-cart-without-wheels.stl"/>
+        <box size ="${base_length} ${base_width} ${base_height}" />
+        <!-- <mesh filename="package://paul_description/meshes/shopping-cart-without-wheels.stl"/> -->
       </geometry>
     </collision>
@@ -139,10 +139,10 @@
   </joint>
   <!-- Arm: xacro must be after so the baseArm joint exists -->
-  <joint name="baseArm" type="fixed">
+  <!-- <joint name="baseArm" type="fixed">
     <parent link="linearAxis_link"/>
     <child link="$(arg arm)_$(arg gripper)_base_link"/>
     <origin xyz="0.0 0.0 0.0" rpy="0 1.5708 0"/>
   </joint>
-  <xacro:include filename="$(find paul_description)/urdf/arms/arm.xacro"/>
+  <xacro:include filename="$(find paul_description)/urdf/arms/arm.xacro"/> -->
   <!-- driven wheels -->
     <!-- Right Wheel: "wheel_R_link" and "wheel_R_joint" -->

Commit message: Testbench simulation: - Added custom sun model for proper lighting - Added launch file to start the arm simulation

File: paul/paul_description/urdf/paul.urdf.xacro (robot description, xacro)
@@ -92,6 +92,6 @@
       <origin xyz="0.0 0.0 ${base_height/2}" rpy="0.0 0.0 0.0"/>
       <geometry>
-        <box size ="${base_length} ${base_width} ${base_height}" />
-        <!-- <mesh filename="package://paul_description/meshes/shopping-cart-without-wheels.stl"/> -->
+        <!-- <box size ="${base_length} ${base_width} ${base_height}" /> -->
+        <mesh filename="package://paul_description/meshes/shopping-cart-without-wheels.stl"/>
       </geometry>
     </collision>

Commit message: Added ODrives to robot: - control.launch to start elevation and propulsion - Added elevationJoint to URDF - Added README to paul_control and removed scripts - Single yaml file to configure controllers - odrives.yaml with the ODrives' configuration - Started updating paul.launch

File: paul/paul_description/urdf/paul.urdf.xacro (robot description, xacro)
@@ -173,5 +173,13 @@
   <!-- ==================== ARM ===================== -->
   <!-- ============================================== -->
-  <xacro:unless value="$(arg sim)">
+  <!-- joint for elevation system motor -->
+  <link name="elevation_motor_link" />
+  <joint name="elevation_motor_joint" type="continuous">
+    <parent link="base_link"/>
+    <child link="elevation_motor_link"/>
+    <axis xyz="0 1 0"/>
+  </joint>
+  <!-- temporary fix to avoid loading the arm -->
+  <xacro:if value="$(arg sim)">
     <!-- linear axis -->
     <link name="linear_axis_link" />
@@ -192,4 +200,4 @@
       <origin xyz="0.0 0.0 0.0" rpy="0.0 0.0 0.0"/>
     </joint>
-  </xacro:unless>
+  </xacro:if>
 </robot>

Commit message: fixed launch files

File: paul/paul_description/urdf/paul.urdf.xacro (robot description, xacro)
@@ -27,5 +27,5 @@
   <xacro:property name="front_to_rear_wheels_x"	value="0.77"/>
   <xacro:property name="front_right_left_y"	value="0.245"/>
-  <xacro:property name="rear_right_left_y"	value="0.22938"/>
+  <xacro:property name="rear_right_left_y"	value="0.559"/>
   <!-- Constant for driven wheels -->
     <!-- Right wheel parameters -->
@@ -154,5 +154,5 @@
   <!-- Lidar sensor -->
   <xacro:lidar parent="base_link">
-    <origin xyz="0.546 0 -0.001" rpy="0 0 0" />
+    <origin xyz="0.546 0 -0.001" rpy="0 0 3.14159" />
   </xacro:lidar>
   <!-- D435 RGB-D Sensor -->
